File: Placas/GateDriver/GateDriver.kicad_sch (KiCad schematic)
At the start: 30 parts, among them J1 Conn_02x04_Odd_Even, J2 Conn_02x04_Odd_Even, Q1 BD135, Q2 BD136, U1 74HC14, U2 LM7815_TO220, U3 HCPL-3120

Commit message: Atualização0.1
Parts:
- R1: value 1k -> 4.7k
- R2: value 10k -> 51k
Changed lines of the file:
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@@
       (effects (font (size 1.27 1.27)))
     )
-    (property "Value" "1k" (at 30.48 41.91 90)
+    (property "Value" "4.7k" (at 30.48 41.91 90)
       (effects (font (size 1.27 1.27)))
     )
@@
       (effects (font (size 1.27 1.27)) (justify right))
     )
-    (property "Value" "10k" (at 95.25 101.6 0)
+    (property "Value" "51k" (at 95.25 101.6 0)
       (effects (font (size 1.27 1.27)) (justify right))
     )

Commit message: Working
Parts:
- removed unit 6 of U1
- removed unit 5 of U1
- removed unit 4 of U1
- removed unit 3 of U1
- R1: value 4.7k -> 1k
Other:
- moved on the sheet: U1B
