File: Placas/Instrumentação/Instrumentação.kicad_pcb (KiCad board)
At the start: 2 copper layers, 95 x 90 mm, 51 parts, among them J1 Conn_01x04_Pin, J2 Conn_02x10_Odd_Even, J3 Conn_01x18_Pin, SW1 SW_Push, U1 TL084, U2 AMS1117-3.3, U3 LA 25-NP, U4 STM32F103C_8-B_Tx

Commit message: Working
Parts:
- added R10: 330, Resistor_THT:R_Axial_DIN0204_L3.6mm_D1.6mm_P7.62mm_Horizontal, F.Cu at (84.2, 89.8)
- renumbered C5 to C4, C6 to C5, C4 to C6, D8 to D6, D6 to D7, D7 to D8, R10 to R11, R11 to R12, R12 to R13, R13 to R14, R14 to R15, R15 to R16
Routing:
- net 3.3V: track 83.4 -> 88.2 mm
